File: Hardware/ESP32-Function.brd (EAGLE design)
At the start: 65 x 38.1 mm, 46 parts, among them J1 MICROMOD_STANDARD, Q2 MBT3904DW1T1, U1 EEPROM, U2 ESP-WROOM-3232D-NARROW, U3 3.3V, U4 CP210X

Commit message: Updates the design to use the Micromod-function device in the official SFE Eagle Libs
Parts:
- J1: value MICROMOD_STANDARD -> MICROMOD_FUNCTION_STANDARD; device SparkFun-MicroMod-Function:M.2-CARD-E-22_FUNCTION_STANDARD -> SparkFun-MicroMod:M.2-CARD-E-22_FUNCTION_STANDARD
Changed lines of the file:
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@@
 <?xml version="1.0" encoding="utf-8"?>
 <!DOCTYPE eagle SYSTEM "eagle.dtd">
-<eagle version="9.6.2">
+<eagle version="9.5.1">
 <drawing>
 <settings>
@@
 <attribute name="REV" value="" x="19.05" y="-11.43" size="1.778" layer="27" font="vector" ratio="15" display="off"/>
 </element>
-<element name="J1" library="SparkFun-MicroMod-Function" package="M.2-CARD-E-22_FUNCTION_STANDARD" value="MICROMOD_STANDARD" x="-0.0118" y="19.016" smashed="yes" rot="R270"/>
+<element name="J1" library="SparkFun-MicroMod" package="M.2-CARD-E-22_FUNCTION_STANDARD" value="MICROMOD_FUNCTION_STANDARD" x="-0.0118" y="19.016" smashed="yes" rot="R270"/>
 <element name="R2" library="SparkFun-Resistors" package="0603" value="10k" x="55.9054" y="36.5252" smashed="yes" rot="R180">
 <attribute name="NAME" x="55.9054" y="35.7632" size="0.6096" layer="25" font="vector" ratio="20" rot="R180" align="bottom-center"/>
