File: Hardware/ESP32-Function.sch (EAGLE design)
At the start: 36 parts, among them J1 MICROMOD_STANDARD, Q2 MBT3904DW1T1, U1 EEPROM, U2 ESP-WROOM-3232D-NARROW, U3 3.3V, U4 CP210X

Commit message: Updates the design to use the Micromod-function device in the official SFE Eagle Libs
Parts:
- J1: value MICROMOD_STANDARD -> MICROMOD_FUNCTION_STANDARD; device SparkFun-MicroMod-Function:MICROMOD_STANDARD -> SparkFun-MicroMod:MICROMOD_FUNCTION_STANDARD
Changed lines of the file:
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@@
 <?xml version="1.0" encoding="utf-8"?>
 <!DOCTYPE eagle SYSTEM "eagle.dtd">
-<eagle version="9.6.2">
+<eagle version="9.5.1">
 <drawing>
 <settings>
@@
 <part name="FRAME2" library="SparkFun-Aesthetics" deviceset="FRAME-LEDGER" device=""/>
 <part name="SUPPLY1" library="SparkFun-PowerSymbols" deviceset="VCC" device=""/>
-<part name="J1" library="SparkFun-MicroMod-Function" deviceset="MICROMOD" device="_STANDARD" value="MICROMOD_STANDARD"/>
+<part name="J1" library="SparkFun-MicroMod" deviceset="MICROMOD_FUNCTION" device="_STANDARD" value="MICROMOD_FUNCTION_STANDARD"/>
 <part name="GND1" library="SparkFun-PowerSymbols" deviceset="GND" device=""/>
 <part name="R2" library="SparkFun-Resistors" deviceset="10KOHM" device="-0603-1/10W-1%" value="10k"/>
